File: basis_a.sch (KiCad schematic (older format))
At the start: 24 parts, among them SW1 SW_Push, U1 ATmega32U4-AU, Y1 16MHz

Commit message: l schema and pcb ver 1 ready
Parts:
- added D? (x29): D_Small, Diode_SMD:D_SOD-123, symbol Device:D_Small
- added MX? (x27): MX-NoLED, MX_Alps_Hybrid:MX-1U-NoLED, symbol MX_Alps_Hybrid:MX-NoLED
- added SW? (x3): Rotary_Encoder_Switch, symbol Device:Rotary_Encoder_Switch
- C4: value .01uF -> 10uF
Connections:
- net COL0: now also SW?.S1, SW?.S1, SW?.S1; no longer MX1.1 (COL), MX2.1 (COL)
- net COL1: now also MX?.1 (COL), MX?.1 (COL), MX?.1 (COL), MX?.1 (COL), MX?.1 (COL); no longer MX3.1 (COL), MX4.1 (COL)
- net GND: now also SW?.C, SW?.C, SW?.C
- net ROW0: now also D?.1 (K), D?.1 (K), D?.1 (K)
- net ROW1: now also D?.1 (K), D?.1 (K), D?.1 (K)
- new net: D?.2 (A), SW?.S2 (x3)
- new net: D?.2 (A), MX?.2 (ROW) (x25)
- new net: D?.2 (A), MX?.2 (ROW), MX?.2 (ROW)
- new net COL2: MX1.1 (COL), MX2.1 (COL), MX?.1 (COL), MX?.1 (COL), MX?.1 (COL)
- new net COL3: MX3.1 (COL), MX4.1 (COL), MX?.1 (COL), MX?.1 (COL), MX?.1 (COL)
- new net COL4: MX?.1 (COL), MX?.1 (COL), MX?.1 (COL), MX?.1 (COL), MX?.1 (COL)
- new net COL5: MX?.1 (COL), MX?.1 (COL), MX?.1 (COL), MX?.1 (COL), MX?.1 (COL)
- new net COL6: MX?.1 (COL), MX?.1 (COL), MX?.1 (COL), MX?.1 (COL), MX?.1 (COL)
- new net ROT0A: SW?.A
- new net ROT0B: SW?.B
- new net ROT1A: SW?.A
- new net ROT1B: SW?.B
- new net ROT2A: SW?.A
- new net ROT2B: SW?.B
- new net ROW2: D?.1 (K), D?.1 (K), D?.1 (K), D?.1 (K), D?.1 (K)
- new net ROW3: D?.1 (K), D?.1 (K), D?.1 (K), D?.1 (K)
- new net ROW4: D?.1 (K), D?.1 (K), D?.1 (K), D?.1 (K), D?.1 (K), D?.1 (K)
Other:
- moved on the sheet: D1, D2, D3, D4, MX1, MX2, MX3, MX4
