File: basis_combined_PROTON.kicad_pcb (KiCad board)
At the start: 2 copper layers, 160.3 x 94.5 mm, 146 parts, among them J1 AudioJack4, J2 AudioJack4, SW1 Rotary_Encoder_Switch, SW2 Rotary_Encoder_Switch, SW3 Rotary_Encoder_Switch, U1 proton_c, U2 proton_c

Commit message: done with usbs
Parts:
- added C1: 10uf, Capacitor_SMD:C_0805_2012Metric, B.Cu at (56.4, 30.2)
- added C10: 22uF, Capacitor_SMD:C_0805_2012Metric, B.Cu at (184.9, 158.8)
- added C11: 22uF, Capacitor_SMD:C_0805_2012Metric, B.Cu at (184.9, 166.7)
- added C12: 0.1uF, Capacitor_SMD:C_0805_2012Metric, B.Cu at (174.6, 186.5)
- added C13: 0.1uf, Capacitor_SMD:C_0805_2012Metric, B.Cu at (158.0, 178.6)
- added C14: 0.1uf, Capacitor_SMD:C_0805_2012Metric, B.Cu at (161.1, 172.2)
- added C15: 1uF, Capacitor_SMD:C_0805_2012Metric, B.Cu at (177.8, 173.8)
- added C16: 0.1uf, Capacitor_SMD:C_0805_2012Metric, B.Cu at (164.3, 190.5)
- added C2: 22uF, Capacitor_SMD:C_0805_2012Metric, B.Cu at (71.4, 46.8)
- added C3: 22uF, Capacitor_SMD:C_0805_2012Metric, B.Cu at (71.4, 38.9)
- added C4: 0.1uF, Capacitor_SMD:C_0805_2012Metric, B.Cu at (58.7, 57.9)
- added C5: 0.1uf, Capacitor_SMD:C_0805_2012Metric, B.Cu at (76.2, 64.3)
- added C6: 0.1uf, Capacitor_SMD:C_0805_2012Metric, B.Cu at (67.5, 31.0)
- added C7: 1uF, Capacitor_SMD:C_0805_2012Metric, B.Cu at (64.3, 30.2)
- added C8: 0.1uf, Capacitor_SMD:C_0805_2012Metric, B.Cu at (66.7, 73.0)
- added C9: 10uf, Capacitor_SMD:C_0805_2012Metric, B.Cu at (165.9, 132.6)
- added F1: 500mA, Fuse:Fuse_1206_3216Metric, B.Cu at (55.6, 26.2)
- added F2: 500mA, Fuse:Fuse_1206_3216Metric, B.Cu at (169.1, 130.0)
- added H1: Hole, 3d-split-keeb:MountingHole-m2, F.Cu at (193.7, 134.1)
- added H2: Hole, 3d-split-keeb:MountingHole-m2, F.Cu at (55.6, 151.6)
- added H3: Hole, 3d-split-keeb:MountingHole-m2, F.Cu at (154.8, 196.8)
- added H4: Hole, 3d-split-keeb:MountingHole-m2, F.Cu at (74.6, 189.7)
- added H5: Hole, 3d-split-keeb:MountingHole-m2, F.Cu at (158.8, 90.5)
- added H6: Hole, 3d-split-keeb:MountingHole-m2, F.Cu at (177.8, 52.4)
- added H7: Hole, 3d-split-keeb:MountingHole-m2, F.Cu at (39.7, 34.9)
- added H8: Hole, 3d-split-keeb:MountingHole-m2, F.Cu at (78.6, 97.6)
- added J3: USB_B_Micro, Connector_USB:USB_Micro-B_Molex_47346-0001, B.Cu at (61.1, 16.9)
- added J4: USB_B_Micro, Connector_USB:USB_Micro-B_Molex_47346-0001, B.Cu at (172.2, 116.2)
- added R10: 22, Resistor_SMD:R_0805_2012Metric, B.Cu at (173.0, 139.7)
- added R11: 10k, Resistor_SMD:R_0805_2012Metric, B.Cu at (177.8, 184.2)
- added R12: 10k, Resistor_SMD:R_0805_2012Metric, B.Cu at (162.1, 192.2)
- added R5: 22, Resistor_SMD:R_0805_2012Metric, B.Cu at (59.5, 25.4)
- added R6: 22, Resistor_SMD:R_0805_2012Metric, B.Cu at (61.9, 25.4)
- added R7: 10k, Resistor_SMD:R_0805_2012Metric, B.Cu at (70.6, 24.6)
- added R8: 10k, Resistor_SMD:R_0805_2012Metric, B.Cu at (66.7, 77.8)
- added R9: 22, Resistor_SMD:R_0805_2012Metric, B.Cu at (170.7, 139.7)
- added SW4: SW_Push, random-keyboard-parts:SKQG-1155865, B.Cu at (72.2, 18.3)
- added SW5: SW_Push, random-keyboard-parts:SKQG-1155865, B.Cu at (181.8, 181.8)
- added Y1: Crystal_GND24_Small, Crystal:Crystal_SMD_3225-4Pin_3.2x2.5mm, B.Cu at (71.4, 42.9)
- added Y2: Crystal_GND24_Small, Crystal:Crystal_SMD_3225-4Pin_3.2x2.5mm, B.Cu at (184.9, 162.7)
- J1: value AudioJack4 -> USB_B_Micro; footprint Keebio-Parts:TRRS-PJ-320A -> Connector_USB:USB_Micro-B_Molex_47346-0001
- J2: value AudioJack4 -> USB_B_Micro; footprint Keebio-Parts:TRRS-PJ-320A -> Connector_USB:USB_Micro-B_Molex_47346-0001; moved to B.Cu
- R3, R4: moved to B.Cu
- SW1, SW2, SW3: footprint Rotary_Encoder:RotaryEncoder_Alps_EC11E-Switch_Vertical_H20mm -> 3d-split-keeb:Rotary_encoder_switch_HOTSWAP
- U1, U2: value proton_c -> ATmega32U4-AU; footprint proton_c:proton_c -> Package_QFP:TQFP-44_10x10mm_P0.8mm
- moved R3 103.0 mm to (172.2, 193.0), turned to 90 degrees
- moved R4 96.7 mm to (169.9, 193.7), turned to 90 degrees
- moved J1 77.8 mm to (177.8, 16.9), turned to 0 degrees
- moved J2 74.8 mm to (55.6, 116.1)
- moved U2 53.4 mm to (166.7, 181.8), turned to 225 degrees
- moved MXsp_rC1 28.6 mm to (55.6, 199.2), turned to 180 degrees
- moved U1 27.8 mm to (67.5, 61.9), turned to 315 degrees
- moved D43 18.1 mm to (73.0, 193.7)
- moved D38 14.3 mm to (42.1, 192.1)
- moved D39 12.3 mm to (64.3, 117.5)
- moved D34 11.7 mm to (42.1, 115.9), turned to 180 degrees
- moved D35 11.7 mm to (42.1, 134.9), turned to 180 degrees
- moved D36 11.7 mm to (42.1, 154.0), turned to 180 degrees
- moved D37 11.4 mm to (42.1, 173.0), turned to 180 degrees
- moved R2 9.59 mm to (73.0, 27.8)
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Connections:
- D6 pad 1: ROW1 -> ROW3
- D7 pad 1: ROW2 -> ROW4
- MX\1 pad 1: COL12 -> COL13
- MX]1 pad 1: COL12 -> COL13
- MX`=1 pad 1: COL12 -> COL13
- MXdel1 pad 1: COL12 -> COL13
- MXret1 pad 1: COL12 -> COL13
- MXspC1 pad 2: Net-(D28-Pad2) -> Net-(D29-Pad2)
- MXsp_rC1 pad 1: COL8 -> COL7
- R1 pad 1: VCC -> TRRS1
- R1 pad 2: TRRS0 -> +5V
- R2 pad 1: TRRS1 -> TRRS0
- R2 pad 2: VCC -> +5V
- R3 pad 1: VCC -> +5V
- R4 pad 1: TRRS1_r -> +5V
- R4 pad 2: VCC -> TRRS1_r
Routing:
- net GND: track 140.7 -> 680.9 mm, vias 0 -> 12
- net +5V: track 49.8 -> 548.7 mm, vias 0 -> 14
- net COL7: track 0.00 -> 253.2 mm, vias 0 -> 11
- net COL8: track 0.00 -> 226.8 mm, vias 0 -> 11
- net TRRS0_r: track 0.00 -> 203.6 mm, vias 0 -> 6
- net TRRS1_r: track 0.00 -> 199.1 mm, vias 0 -> 6
- net COL9: track 0.00 -> 188.0 mm, vias 0 -> 8
- net COL10: track 0.00 -> 182.9 mm, vias 0 -> 11
- net COL11: track 0.00 -> 160.4 mm, vias 0 -> 11
- net COL13: track 0.00 -> 134.2 mm, vias 0 -> 6
- net ROW9: track 74.6 -> 202.7 mm, vias 0 -> 3
- net COL12: track 0.32 -> 119.7 mm, vias 0 -> 8
- net TRRS0: track 47.3 -> 148.8 mm, vias 1 -> 4
- net TRRS1: track 45.4 -> 146.5 mm, vias 1 -> 4
- net ROW8: track 99.2 -> 199.9 mm, vias 0 -> 6
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- added copper zone on B.Cu, net GND
Other:
- board size 160.3 x 94.5 mm -> 160.3 x 193.7 mm
- board text added: "basis 0.0.1"

Commit message: version sent to pcb manu
Parts:
- J1, J2, J3, J4: footprint Connector_USB:USB_Micro-B_Molex_47346-0001 -> Connector_USB:USB_Micro-B_Molex-105017-0001
- moved C1 188.6 mm to (-104.0, 129.4)
- moved C2 188.6 mm to (-88.9, 146.1)
- moved C3 188.6 mm to (-88.9, 138.1)
- moved C5 188.6 mm to (-84.1, 163.5)
- moved C6 188.6 mm to (-92.9, 130.2)
- moved C7 188.6 mm to (-96.0, 129.4)
- moved D1 188.6 mm to (-57.1, 117.5)
- moved D10 188.6 mm to (-81.0, 155.6)
- moved D11 188.6 mm to (-81.0, 174.6)
- moved D12 188.6 mm to (-76.2, 193.7)
- moved D13 188.6 mm to (-57.1, 155.6)
- moved D14 188.6 mm to (-57.1, 174.6)
- moved D15 188.6 mm to (-57.1, 193.7)
- moved D16 188.6 mm to (-38.1, 155.6)
- moved D17 188.6 mm to (-38.1, 174.6)
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Connections:
- J2 pad 2: TRRS1_r -> TRRS1
- J2 pad 3: TRRS0_r -> TRRS0
- R3 pad 2: TRRS0_r -> TRRS0
- R4 pad 2: TRRS1_r -> TRRS1
- U2 pad 18: TRRS0_r -> TRRS0
- U2 pad 19: TRRS1_r -> TRRS1
Routing:
- net TRRS0: track 148.8 -> 393.0 mm, vias 4 -> 12
- net TRRS1: track 146.5 -> 386.4 mm, vias 4 -> 12
- net TRRS0_r: track 203.6 -> 0.00 mm, vias 6 -> 0
- net TRRS1_r: track 199.1 -> 0.00 mm, vias 6 -> 0
- net GND: track 680.9 -> 736.2 mm, vias 12 -> 15
- net +5V: track 548.7 -> 598.8 mm, vias 14 -> 17
- net Net-(D63-Pad2): track 0.00 -> 15.3 mm
- net COL6: track 260.6 -> 273.7 mm
- net COL9: track 188.0 -> 182.7 mm
- net COL10: track 182.9 -> 177.6 mm
- net COL8: track 226.8 -> 221.6 mm
- net Net-(D68-Pad2): track 8.80 -> 14.1 mm
- net COL11: track 160.4 -> 156.4 mm
- net COL7: track 253.2 -> 249.2 mm
- net COL5: track 234.8 -> 232.3 mm
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Other:
- board size 160.3 x 193.7 mm -> 320.7 x 94.5 mm

Commit message: missed files? don't know'
Parts:
- added D69: WS2813, LED_SMD:LED_WS2812_PLCC6_5.0x5.0mm_P1.6mm, F.Cu at (-76.0, 141.9)
- D1, D10, D11, D12, D13, D14, D15, D16, D17, D18, D19, D2, D20, D21, D22, D23, D24, D25, D26, D27, D28, D29, D3, D30, D31, D32, D33, D34, D35, D36, D37, D38, D39, D4, D40, D41, D42, D43, D44, D45, D46, D47, D48, D49, D5, D50, D51, D52, D53, D54, D55, D56, D57, D58, D59, D6, D60, D61, D62, D63, D64, D65, D66, D67, D68, D7, D8, D9: footprint Diode_SMD:D_SOD-123 -> Diode_SMD:D_SOD-323F
- moved D10 0.89 mm to (-81.0, 156.5)
- moved D11 0.51 mm to (-81.0, 174.1)
- moved D12 0.51 mm to (-76.2, 193.2)
- moved D14 0.51 mm to (-57.1, 174.1)
- moved D15 0.51 mm to (-57.1, 193.2)
- moved D17 0.51 mm to (-38.1, 174.1)
- moved D18 0.51 mm to (-38.1, 193.2)
- moved D2 0.51 mm to (-57.1, 136.0)
- moved D20 0.51 mm to (-19.1, 136.0)
- moved D22 0.51 mm to (-19.1, 174.1)
- moved D23 0.51 mm to (-19.1, 193.2)
- moved D25 0.51 mm to (0.00, 136.0)
- moved D27 0.51 mm to (0.00, 174.1)
- moved D28 0.51 mm to (0.00, 193.2)
- moved D31 0.51 mm to (19.1, 136.0)
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Routing:
- net GND: track 736.2 -> 747.3 mm, vias 15 -> 16
- net Net-(D49-Pad2): track 13.7 -> 17.8 mm
- net Net-(D13-Pad2): track 13.6 -> 17.7 mm
- net Net-(D42-Pad2): track 13.1 -> 17.2 mm
- net Net-(D64-Pad2): track 13.7 -> 17.7 mm
- net Net-(D54-Pad2): track 13.7 -> 17.7 mm
- net Net-(D59-Pad2): track 13.7 -> 17.7 mm
- net Net-(D47-Pad2): track 13.8 -> 17.7 mm
- net Net-(D44-Pad2): track 13.9 -> 17.7 mm
- net Net-(D34-Pad2): track 15.6 -> 18.5 mm
- net Net-(D20-Pad2): track 14.9 -> 17.8 mm
- net Net-(D19-Pad2): track 14.9 -> 17.7 mm
- net Net-(D9-Pad2): track 14.9 -> 17.7 mm
- net Net-(D2-Pad2): track 14.9 -> 17.7 mm
- net Net-(D4-Pad2): track 14.9 -> 17.7 mm
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
Commit message: Added a bunch of cleanup etc
Parts:
- removed D69: WS2813, LED_SMD:LED_WS2812_PLCC6_5.0x5.0mm_P1.6mm
- added U3: SRV05-4, Package_TO_SOT_SMD:SOT-23-6, B.Cu at (-101.2, 136.9)
- added U4: SRV05-4, Package_TO_SOT_SMD:SOT-23-6, B.Cu at (56.0, 122.2)
- added U5: SRV05-4, Package_TO_SOT_SMD:SOT-23-6, B.Cu at (17.5, 122.2)
- added U6: SRV05-4, Package_TO_SOT_SMD:SOT-23-6, B.Cu at (171.8, 137.7)
- C10, C11, C2, C3: value 22uF -> 22pF
- moved R4 95.2 mm to (97.2, 132.2), turned to 180 degrees
- moved R3 93.2 mm to (101.6, 132.2), turned to 0 degrees
- moved C10 35.5 mm to (172.6, 192.1), turned to 315 degrees
- moved Y2 29.1 mm to (175.0, 190.1), turned to 45 degrees
- moved SW5 24.4 mm to (184.9, 157.6), turned to 90 degrees
- moved C7 22.7 mm to (-98.4, 152.0)
- moved C11 22.6 mm to (177.1, 187.9), turned to 135 degrees
- moved R11 22.5 mm to (185.7, 163.1), turned to 180 degrees
- moved R5 21.5 mm to (-102.4, 146.1)
- moved R6 21.5 mm to (-100.0, 146.1)
- moved C6 19.1 mm to (-93.8, 149.2), turned to 180 degrees
- moved C3 14.8 mm to (-87.3, 152.8), turned to 0 degrees
- moved D43 8.33 mm to (64.7, 193.2)
- moved Y1 7.71 mm to (-87.3, 149.6), turned to 270 degrees
- moved D5 7.53 mm to (-113.5, 134.1), turned to 90 degrees
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Routing:
- net COL13: track 134.2 -> 183.6 mm, vias 6 -> 1
- net Net-(C10-Pad1): track 46.4 -> 8.29 mm
- net Net-(C11-Pad1): track 49.5 -> 12.5 mm, vias 2 -> 0
- net +5V: track 599.7 -> 630.7 mm, vias 17 -> 23
- net Net-(C7-Pad1): track 32.4 -> 5.46 mm
- net D+: track 27.9 -> 54.8 mm
- net D-: track 29.1 -> 55.4 mm
- net COL6: track 273.7 -> 248.7 mm, vias 0 -> 1
- net COL10: track 177.6 -> 201.0 mm, vias 11 -> 3
- net COL8: track 221.6 -> 244.9 mm, vias 11 -> 3
- net COL7: track 249.2 -> 271.5 mm, vias 11 -> 3
- net COL9: track 182.7 -> 204.5 mm, vias 8 -> 1
- net COL11: track 156.4 -> 177.5 mm, vias 11 -> 3
- net Net-(R6-Pad1): track 33.5 -> 12.8 mm
- net Net-(R5-Pad1): track 34.2 -> 13.5 mm
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- added copper zone on F.Cu, net GND
Other:
- outline, holes or cut-outs redrawn
- board text added: "basis 0.0.2"
- board text removed: "basis 0.0.1"

Commit message: checkpoint
Parts:
- removed D19, D20, D21, D22, D23, D24, D25, D26, D27, D28, D29, D30, D31, D32, D33: D_Small, Diode_SMD:D_SOD-323F
- added H9: Hole, 3d-split-keeb:MountingHole-m2, F.Cu at (-115.9, 166.7)
- added R13: 4.7k, Resistor_SMD:R_0805_2012Metric, B.Cu at (-100.0, 119.9)
- added R14: 4.7k, Resistor_SMD:R_0805_2012Metric, B.Cu at (-94.5, 119.9)
- added R15: 4.7k, Resistor_SMD:R_0805_2012Metric, B.Cu at (161.9, 114.7)
- added R16: 4.7k, Resistor_SMD:R_0805_2012Metric, B.Cu at (179.0, 115.1)
- D1, D10, D11, D12, D13, D14, D15, D16, D17, D18, D2, D3, D4, D8, D9: value D_Small -> D_Schottky_x2_KCom_AAK; footprint Diode_SMD:D_SOD-323F -> 3d-split-keeb:D_SOT-23_AAK
- J1, J2: footprint Connector_USB:USB_Micro-B_Molex-105017-0001 -> 3d-split-keeb:MOLEX_47642-0001-fixed
- J3, J4: value USB_B_Micro -> USB_C_Receptacle_USB2.0; footprint Connector_USB:USB_Micro-B_Molex-105017-0001 -> random-keyboard-parts:USB_C_Receptacle_Hirose_CX90M-16P
- MX'1, MX,1, MX.1, MX/1, MX0, MX1, MX2, MX3, MX4, MX5, MX6, MX7, MX8, MX9, MX;1, MX\1, MX]1, MX`-1, MX`1, MX`=1, MXa1, MXb1, MXc1, MXcm1, MXct1, MXd1, MXdel1, MXdown1, MXe1, MXes1, MXf1, MXfn1, MXg1, MXh1, MXi1, MXj1, MXk1, MXl1, MXleft1, MXm1, MXn1, MXo1, MXop1, MXp1, MXq1, MXr1, MXret1, MXright1, MXs1, MXsh1, MXsh_r1, MXsp0, MXsp1, MXspC1, MXsp_r0, MXsp_r1, MXsp_rC1, MXt1, MXtb1, MXtb[1, MXu1, MXup1, MXv1, MXw1, MXx1, MXy1, MXz1: footprint 3d-split-keeb:Kailh_socket_MX_optional_FLIPPED -> 3d-split-keeb:Kailh_socket_MX_optional_FLIPPED_PTH
- SW4, SW5: footprint random-keyboard-parts:SKQG-1155865 -> random-keyboard-parts:KXT-311-LHSSwitch
- moved D15 93.9 mm to (17.5, 136.1), turned to 90 degrees
- moved D14 85.6 mm to (6.35, 116.7), turned to 90 degrees
- moved D8 78.6 mm to (-58.7, 193.3), turned to 90 degrees
- moved D10 64.3 mm to (-20.6, 136.1), turned to 90 degrees
- moved D11 63.2 mm to (-20.6, 155.2), turned to 90 degrees
- moved D9 63.2 mm to (-20.6, 117.1), turned to 90 degrees
- moved D12 58.7 mm to (-20.6, 174.2), turned to 90 degrees
- moved D16 55.6 mm to (17.5, 157.2), turned to 90 degrees
- moved D17 55.6 mm to (17.5, 174.2), turned to 90 degrees
- moved D18 54.0 mm to (15.9, 191.7), turned to 90 degrees
- moved D13 52.9 mm to (-20.6, 193.3), turned to 90 degrees
- moved D4 43.4 mm to (-58.7, 174.2), turned to 90 degrees
- moved D3 43.4 mm to (-58.7, 155.2), turned to 90 degrees
- moved R4 37.7 mm to (134.9, 132.2)
- moved R3 36.9 mm to (138.5, 132.2)
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Connections:
- D1 pad 1: ROW0 -> Net-(D1-Pad1)
- D10 pad 1: ROW2 -> Net-(D10-Pad1)
- D11 pad 1: ROW3 -> Net-(D11-Pad1)
- D12 pad 1: ROW4 -> Net-(D12-Pad1)
- D13 pad 1: ROW2 -> Net-(D13-Pad1)
- D14 pad 1: ROW3 -> Net-(D14-Pad1)
- D15 pad 1: ROW4 -> Net-(D15-Pad1)
- D16 pad 1: ROW2 -> Net-(D16-Pad1)
- D17 pad 1: ROW3 -> Net-(D17-Pad1)
- D18 pad 1: ROW4 -> Net-(D18-Pad1)
- D2 pad 1: ROW1 -> Net-(D2-Pad1)
- D3 pad 1: ROW0 -> Net-(D3-Pad1)
- D4 pad 1: ROW1 -> Net-(D4-Pad1)
- D8 pad 1: ROW0 -> Net-(D8-Pad1)
- D9 pad 1: ROW1 -> Net-(D9-Pad1)
- MX2 pad 1: COL3 -> Net-(D9-Pad1)
- MX2 pad 2: Net-(D3-Pad2) -> COL3
- MX3 pad 2: Net-(D19-Pad2) -> Net-(D9-Pad2)
- MX4 pad 1: COL5 -> Net-(D14-Pad1)
- MX4 pad 2: Net-(D24-Pad2) -> COL5
- MX5 pad 2: Net-(D30-Pad2) -> Net-(D14-Pad2)
- MX`1 pad 1: COL1 -> Net-(D1-Pad1)
- MX`1 pad 2: Net-(D8-Pad2) -> COL1
- MXa1 pad 2: Net-(D13-Pad2) -> Net-(D3-Pad2)
- MXb1 pad 2: Net-(D33-Pad2) -> Net-(D17-Pad2)
- MXc1 pad 2: Net-(D22-Pad2) -> Net-(D12-Pad2)
- MXcm1 pad 2: Net-(D23-Pad2) -> Net-(D13-Pad2)
- MXct1 pad 2: Net-(D15-Pad2) -> Net-(D8-Pad2)
- MXd1 pad 2: Net-(D21-Pad2) -> Net-(D11-Pad2)
- MXe1 pad 2: Net-(D20-Pad2) -> Net-(D10-Pad2)
- MXes1 pad 1: COL1 -> Net-(D3-Pad1)
- MXes1 pad 2: Net-(D10-Pad2) -> COL1
- MXf1 pad 1: COL5 -> Net-(D16-Pad1)
- MXf1 pad 2: Net-(D26-Pad2) -> COL5
- MXfn1 pad 1: COL1 -> Net-(D8-Pad1)
- MXfn1 pad 2: Net-(D12-Pad2) -> COL1
- MXg1 pad 2: Net-(D32-Pad2) -> Net-(D16-Pad2)
- MXop1 pad 1: COL3 -> Net-(D13-Pad1)
- MXop1 pad 2: Net-(D18-Pad2) -> COL3
- MXr1 pad 1: COL5 -> Net-(D15-Pad1)
- MXr1 pad 2: Net-(D25-Pad2) -> COL5
- MXs1 pad 1: COL3 -> Net-(D11-Pad1)
- MXs1 pad 2: Net-(D16-Pad2) -> COL3
- MXsh1 pad 1: COL1 -> Net-(D4-Pad1)
- MXsh1 pad 2: Net-(D11-Pad2) -> COL1
- MXsp0 pad 1: COL5 -> Net-(D18-Pad1)
- MXsp0 pad 2: Net-(D28-Pad2) -> COL5
- MXsp1 pad 1: COL6 -> Net-(D18-Pad2)
- MXsp1 pad 2: Net-(D29-Pad2) -> COL6
- MXspC1 pad 1: COL5 -> Net-(D18-Pad1)
- MXspC1 pad 2: Net-(D29-Pad2) -> COL6
- MXt1 pad 2: Net-(D31-Pad2) -> Net-(D15-Pad2)
- MXtb1 pad 1: COL1 -> Net-(D2-Pad1)
- MXtb1 pad 2: Net-(D9-Pad2) -> COL1
- MXv1 pad 1: COL5 -> Net-(D17-Pad1)
- MXv1 pad 2: Net-(D27-Pad2) -> COL5
- MXw1 pad 1: COL3 -> Net-(D10-Pad1)
- MXw1 pad 2: Net-(D4-Pad2) -> COL3
- MXx1 pad 1: COL3 -> Net-(D12-Pad1)
- MXx1 pad 2: Net-(D17-Pad2) -> COL3
- MXz1 pad 2: Net-(D14-Pad2) -> Net-(D4-Pad2)
- U1 pad 20: COL6 -> Net-(U1-Pad20)
- U1 pad 21: COL5 -> Net-(U1-Pad21)
- U1 pad 25: COL4 -> COL6
- U1 pad 26: COL3 -> COL5
- U1 pad 27: COL2 -> COL4
- U1 pad 28: COL1 -> COL3
- U1 pad 31: Net-(U1-Pad31) -> COL2
- U1 pad 32: Net-(U1-Pad32) -> COL1
- U3 pad 3: D+ -> D-
- U3 pad 4: Net-(U3-Pad4) -> D+
- U3 pad 6: Net-(U3-Pad6) -> D+
- U4 pad 1: Net-(U4-Pad1) -> TRRS0
- U4 pad 3: Net-(U4-Pad3) -> TRRS0
- U4 pad 6: TRRS0 -> TRRS1
- U5 pad 1: Net-(U5-Pad1) -> TRRS0
- U5 pad 3: Net-(U5-Pad3) -> TRRS0
- U5 pad 6: TRRS0 -> TRRS1
- U6 pad 1: Net-(U6-Pad1) -> D+
- U6 pad 3: Net-(U6-Pad3) -> D+
- U6 pad 6: D+ -> D-
Routing:
- net GND: track 748.4 -> 926.4 mm, vias 20 -> 59
- net COL8: track 244.9 -> 195.7 mm
- net COL11: track 177.5 -> 128.6 mm
- net COL10: track 201.0 -> 152.2 mm
- net COL12: track 139.2 -> 90.7 mm
- net COL9: track 204.5 -> 156.0 mm
- net COL13: track 183.6 -> 135.1 mm
- net COL7: track 271.5 -> 233.5 mm
- net COL5: track 235.5 -> 199.5 mm
- net VCC: track 20.6 -> 53.5 mm, vias 0 -> 4
- net COL3: track 188.5 -> 162.7 mm
- net COL1: track 148.9 -> 123.8 mm
- net D+: track 54.8 -> 79.5 mm, vias 0 -> 4
- net D-: track 55.4 -> 80.0 mm, vias 0 -> 4
- net Net-(D18-Pad1): track 0.00 -> 23.8 mm
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Other:
- board size 320.7 x 94.5 mm -> 320.7 x 98.5 mm
