File: basis_combined_PROTON.kicad_pcb (KiCad board)
At the start: 2 copper layers, 320.7 x 98.5 mm, 180 parts, among them J1 USB_B_Micro, J2 USB_B_Micro, J3 USB_C_Receptacle_USB2.0, J4 USB_C_Receptacle_USB2.0, SW1 Rotary_Encoder_Switch, SW2 Rotary_Encoder_Switch, SW3 Rotary_Encoder_Switch, SW4 SW_Push, SW5 SW_Push, U1 ATmega32U4-AU, U2 ATmega32U4-AU, U3 SRV05-4, U4 SRV05-4, U5 SRV05-4, U6 SRV05-4, Y1 Crystal_GND24_Small, Y2 Crystal_GND24_Small

Commit message: Delete some chaff
Parts:
- removed D49, D50, D51, D52, D53, D54, D55, D56, D57, D58, D59, D60, D61, D62, D63: D_Small, Diode_SMD:D_SOD-323F
- removed H2, H6: Hole, 3d-split-keeb:MountingHole-m2
- removed R10, R9: 22, Resistor_SMD:R_0805_2012Metric
- removed R11, R12: 10k, Resistor_SMD:R_0805_2012Metric
- removed SW5: SW_Push, random-keyboard-parts:KXT-311-LHSSwitch
- removed Y1, Y2: Crystal_GND24_Small, Crystal:Crystal_SMD_3225-4Pin_3.2x2.5mm
- added B1: BLUENRG-M2SA, 3d-split-keeb:BLUENRG-M2SA, B.Cu at (-86.1, 195.3)
- added B2: BLUENRG-M2SA, 3d-split-keeb:BLUENRG-M2SA, B.Cu at (167.5, 191.3)
- added C17: 4.7uF, Capacitor_SMD:C_0402_1005Metric, B.Cu at (-95.3, 129.1)
- added C18: 100nF, Capacitor_SMD:C_0402_1005Metric, B.Cu at (-95.3, 130.5)
- added C19: 4.7uF, Capacitor_SMD:C_0402_1005Metric, B.Cu at (-101.4, 126.7)
- added C20: 10nF, Capacitor_SMD:C_0402_1005Metric, B.Cu at (-94.3, 123.3)
- added C21: 4.7uF, Capacitor_SMD:C_0402_1005Metric, B.Cu at (-90.1, 121.5)
- added C22: 100nF, Capacitor_SMD:C_0402_1005Metric, B.Cu at (-88.5, 136.8)
- added C23: 1uF, Capacitor_SMD:C_0402_1005Metric, B.Cu at (-90.5, 141.2)
- added C24: 100nF, Capacitor_SMD:C_0402_1005Metric, B.Cu at (-88.7, 135.0)
- added C25: 10nF, Capacitor_SMD:C_0402_1005Metric, B.Cu at (-91.1, 140.5)
- added C26: 100nF, Capacitor_SMD:C_0402_1005Metric, B.Cu at (-99.8, 137.0)
- added C27: 1uF, Capacitor_SMD:C_0402_1005Metric, B.Cu at (-102.3, 121.7)
- added C28: 1uF, Capacitor_SMD:C_0402_1005Metric, B.Cu at (-102.9, 126.1)
- added C29: 100nF, Capacitor_SMD:C_0402_1005Metric, B.Cu at (-57.6, 124.6)
- added C30: 100nF, Capacitor_SMD:C_0402_1005Metric, B.Cu at (128.2, 194.5)
- added C31: 100nF, Capacitor_SMD:C_0402_1005Metric, B.Cu at (0.40, 124.6)
- added C32: 100nF, Capacitor_SMD:C_0402_1005Metric, B.Cu at (184.2, 179.0)
- added C33: 100nF, Capacitor_SMD:C_0402_1005Metric, B.Cu at (18.7, 162.7)
- added C34: 100nF, Capacitor_SMD:C_0402_1005Metric, B.Cu at (177.7, 132.4)
- added C35: 100nF, Capacitor_SMD:C_0402_1005Metric, B.Cu at (-0.40, 200.8)
- added C36: 100nF, Capacitor_SMD:C_0402_1005Metric, B.Cu at (-57.9, 201.6)
- added C37: 100nF, Capacitor_SMD:C_0402_1005Metric, B.Cu at (-110.7, 177.8)
- added C38: 100nF, Capacitor_SMD:C_0402_1005Metric, B.Cu at (-111.5, 135.7)
- added C39: 10uF, Capacitor_SMD:C_0402_1005Metric, B.Cu at (-100.4, 164.7)
- added C40: 50uF, Capacitor_SMD:C_0402_1005Metric, B.Cu at (-98.4, 167.9)
- added C41: 50nF, Capacitor_SMD:C_0402_1005Metric, B.Cu at (-93.3, 168.3)
- added C42: 250uF, Capacitor_SMD:C_0402_1005Metric, B.Cu at (-96.0, 168.7)
- added C43: 10uF, Capacitor_SMD:C_0402_1005Metric, B.Cu at (150.0, 161.0)
- added C44: 50uF, Capacitor_SMD:C_0402_1005Metric, B.Cu at (150.0, 166.4)
- added C45: 50nF, Capacitor_SMD:C_0402_1005Metric, B.Cu at (152.4, 167.5)
- added C46: 250uF, Capacitor_SMD:C_0402_1005Metric, B.Cu at (154.0, 174.2)
- added D19: 1N4148, Diode_SMD:D_SOD-323F, B.Cu at (-92.9, 120.9)
- added D20: D_Schottky_Small, Diode_SMD:D_SOD-123, B.Cu at (-105.0, 119.8)
- added D21: 1N4148, Diode_SMD:D_SOD-323F, B.Cu at (191.2, 152.5)
- added D22: D_Schottky_Small, Diode_SMD:D_SOD-123, B.Cu at (175.0, 129.1)
- added D23: WS2812B, LED_SMD:LED_WS2812B_PLCC4_5.0x5.0mm_P3.2mm, B.Cu at (131.8, 120.7)
- added D24: WS2812B, LED_SMD:LED_WS2812B_PLCC4_5.0x5.0mm_P3.2mm, B.Cu at (74.6, 120.7)
- added D25: WS2812B, LED_SMD:LED_WS2812B_PLCC4_5.0x5.0mm_P3.2mm, B.Cu at (55.6, 158.8)
- added D26: WS2812B, LED_SMD:LED_WS2812B_PLCC4_5.0x5.0mm_P3.2mm, B.Cu at (74.6, 196.8)
- added D27: WS2812B, LED_SMD:LED_WS2812B_PLCC4_5.0x5.0mm_P3.2mm, B.Cu at (-58.7, 120.7)
- added D28: WS2812B, LED_SMD:LED_WS2812B_PLCC4_5.0x5.0mm_P3.2mm, B.Cu at (131.8, 196.8)
- added D29: WS2812B, LED_SMD:LED_WS2812B_PLCC4_5.0x5.0mm_P3.2mm, B.Cu at (-1.59, 120.6)
- added D30: WS2812B, LED_SMD:LED_WS2812B_PLCC4_5.0x5.0mm_P3.2mm, B.Cu at (180.2, 180.2)
- added D31: WS2812B, LED_SMD:LED_WS2812B_PLCC4_5.0x5.0mm_P3.2mm, B.Cu at (17.5, 158.8)
- added D32: WS2812B, LED_SMD:LED_WS2812B_PLCC4_5.0x5.0mm_P3.2mm, B.Cu at (181.8, 132.6)
- added D33: WS2812B, LED_SMD:LED_WS2812B_PLCC4_5.0x5.0mm_P3.2mm, B.Cu at (-1.59, 196.8)
- added D69: WS2812B, LED_SMD:LED_WS2812B_PLCC4_5.0x5.0mm_P3.2mm, B.Cu at (-58.7, 196.9)
- added D70: WS2812B, LED_SMD:LED_WS2812B_PLCC4_5.0x5.0mm_P3.2mm, B.Cu at (-106.4, 180.2)
- added D71: WS2812B, LED_SMD:LED_WS2812B_PLCC4_5.0x5.0mm_P3.2mm, B.Cu at (-108.7, 132.6)
- added H10: Hole, 3d-split-keeb:Mounting_Wuerth_WA-SMSI-M2_H3.5mm_9774035243, F.Cu at (74.6, 132.6)
- added H7: Hole, 3d-split-keeb:Mounting_Wuerth_WA-SMSI-M2_H3.5mm_9774035243, F.Cu at (-110.7, 167.1)
- added J5: FTSH-105-01-L-DV-K, FTSH-105-01-L-DV-K:SAMTEC_FTSH-105-01-L-DV-K, B.Cu at (-84.9, 117.5)
- added J6: FTSH-105-01-L-DV-K, FTSH-105-01-L-DV-K:SAMTEC_FTSH-105-01-L-DV-K, B.Cu at (153.3, 194.1)
- added J7: FTSH-105-01-L-DV-K, FTSH-105-01-L-DV-K:SAMTEC_FTSH-105-01-L-DV-K, B.Cu at (192.5, 117.9)
- added J8: FTSH-105-01-L-DV-K, FTSH-105-01-L-DV-K:SAMTEC_FTSH-105-01-L-DV-K, B.Cu at (-95.2, 186.1)
- added LS1: Speaker, 3d-split-keeb:cms-151103-16sp, F.Cu at (-82.5, 181.8)
- added LS2: Speaker, 3d-split-keeb:cms-151103-16sp, F.Cu at (171.1, 174.6)
- added Q1: DTC123J, Package_TO_SOT_SMD:SOT-723, B.Cu at (-90.1, 120.1)
- added Q2: DTC123J, Package_TO_SOT_SMD:SOT-723, B.Cu at (191.9, 154.4)
- added R17: 100k, Resistor_SMD:R_0402_1005Metric, B.Cu at (-94.3, 124.3)
- added R18: 1M, Resistor_SMD:R_0402_1005Metric, B.Cu at (-102.3, 120.7)
- added REF**: Stabilizer_MX_2u, keyswitches:Stabilizer_MX_2u, F.Cu at (55.6, 199.2)
- added REF**: Stabilizer_MX_2u, keyswitches:Stabilizer_MX_2u, F.Cu at (17.5, 199.2)
- added SW6: SW_Push, random-keyboard-parts:KXT-311-LHSSwitch, B.Cu at (-90.9, 118.2)
- added U10: STM32F072CBUx, Package_DFN_QFN:QFN-48-1EP_7x7mm_P0.5mm_EP5.6x5.6mm, B.Cu at (181.6, 159.4)
- added U11: USBLC6-2SC6, Package_TO_SOT_SMD:SOT-666, B.Cu at (-97.2, 121.5)
- added U12: USBLC6-2SC6, Package_TO_SOT_SMD:SOT-666, B.Cu at (170.3, 121.4)
- added U7: STM32F072CBUx, Package_DFN_QFN:QFN-48-1EP_7x7mm_P0.5mm_EP5.6x5.6mm, B.Cu at (-94.3, 136.0)
- added U8: SN74LVC1G07DCK3, 3d-split-keeb:SN74LVC1G07DCK3, B.Cu at (132.2, 129.0)
- added U9: XC6206PxxxMR, Package_TO_SOT_SMD:SOT-23, B.Cu at (-102.9, 123.9)
- C1: value 10uf -> 4.7uF; footprint Capacitor_SMD:C_0805_2012Metric -> Capacitor_SMD:C_0402_1005Metric
- C10, C2: value 22pF -> 100nF; footprint Capacitor_SMD:C_0805_2012Metric -> Capacitor_SMD:C_0402_1005Metric
- C11, C3: value 22pF -> 4.7uF; footprint Capacitor_SMD:C_0805_2012Metric -> Capacitor_SMD:C_0402_1005Metric
- C12: value 0.1uF -> 1uF; footprint Capacitor_SMD:C_0805_2012Metric -> Capacitor_SMD:C_0402_1005Metric
- C13, C14, C16, C6: value 0.1uf -> 100nF; footprint Capacitor_SMD:C_0805_2012Metric -> Capacitor_SMD:C_0402_1005Metric
- C15: value 1uF -> 100nF; footprint Capacitor_SMD:C_0805_2012Metric -> Capacitor_SMD:C_0402_1005Metric
- C4: value 0.1uF -> 100nF; footprint Capacitor_SMD:C_0805_2012Metric -> Capacitor_SMD:C_0402_1005Metric
- C5: value 0.1uf -> 1uF; footprint Capacitor_SMD:C_0805_2012Metric -> Capacitor_SMD:C_0402_1005Metric
- C7: footprint Capacitor_SMD:C_0805_2012Metric -> Capacitor_SMD:C_0402_1005Metric
- C8: value 0.1uf -> 10nF; footprint Capacitor_SMD:C_0805_2012Metric -> Capacitor_SMD:C_0402_1005Metric
- C9: value 10uf -> 10nF; footprint Capacitor_SMD:C_0805_2012Metric -> Capacitor_SMD:C_0402_1005Metric
- D34, D35, D36, D37, D38, D39, D40, D41, D42, D43, D44, D45, D46, D47, D48: value D_Small -> D_Schottky_x2_KCom_AAK; footprint Diode_SMD:D_SOD-323F -> 3d-split-keeb:D_SOT-23_AAK
- H1, H3, H4, H5, H7, H8, H9: footprint 3d-split-keeb:MountingHole-m2 -> 3d-split-keeb:Mounting_Wuerth_WA-SMSI-M2_H3.5mm_9774035243
- R1: value 4.7k -> 1M; footprint Resistor_SMD:R_0805_2012Metric -> Resistor_SMD:R_0402_1005Metric
- R13, R14, R15, R16, R2, R3: footprint Resistor_SMD:R_0805_2012Metric -> Resistor_SMD:R_0402_1005Metric
- R4: value 4.7k -> 100k; footprint Resistor_SMD:R_0805_2012Metric -> Resistor_SMD:R_0402_1005Metric
- R5: value 22 -> 1.2k; footprint Resistor_SMD:R_0805_2012Metric -> Resistor_SMD:R_0402_1005Metric
- R6: value 22 -> 10; footprint Resistor_SMD:R_0805_2012Metric -> Resistor_SMD:R_0402_1005Metric
- R7: value 10k -> 1.2k; footprint Resistor_SMD:R_0805_2012Metric -> Resistor_SMD:R_0402_1005Metric
- R8: value 10k -> 10; footprint Resistor_SMD:R_0805_2012Metric -> Resistor_SMD:R_0402_1005Metric
- U1: value ATmega32U4-AU -> SN74LVC1G07DCK3; footprint Package_QFP:TQFP-44_10x10mm_P0.8mm -> 3d-split-keeb:SN74LVC1G07DCK3
- U2: value ATmega32U4-AU -> XC6206PxxxMR; footprint Package_QFP:TQFP-44_10x10mm_P0.8mm -> Package_TO_SOT_SMD:SOT-23
- U3, U6: value SRV05-4 -> LM386; footprint Package_TO_SOT_SMD:SOT-23-6 -> Package_SO:SOIC-8_3.9x4.9mm_P1.27mm
- moved C1 286.4 mm to (179.8, 153.1), turned to 225 degrees
- moved C8 283.4 mm to (189.0, 152.5), turned to 90 degrees
- moved SW4 282.3 mm to (190.9, 150.5), turned to 180 degrees
- moved C4 277.7 mm to (176.0, 160.4), turned to 315 degrees
- moved C2 274.7 mm to (187.1, 158.3), turned to 135 degrees
- moved C6 274.4 mm to (180.5, 153.8), turned to 225 degrees
- moved C7 272.3 mm to (172.9, 128.5)
- moved C5 269.0 mm to (185.2, 164.4)
- moved C3 267.0 mm to (179.7, 150.1), turned to 90 degrees
- moved R1 258.6 mm to (172.9, 127.5), turned to 180 degrees
- moved R8 248.1 mm to (154.3, 167.5), turned to 180 degrees
- moved R7 243.1 mm to (150.0, 159.1)
- moved C15 120.2 mm to (56.8, 162.7), turned to 180 degrees
- moved C14 100.0 mm to (75.8, 124.6), turned to 180 degrees
- moved C16 89.1 mm to (75.8, 200.8), turned to 180 degrees
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Connections:
- C1 pad 1: +5V -> +3V3
- C10 pad 1: Net-(C10-Pad1) -> +3V3
- C11 pad 1: Net-(C11-Pad1) -> NRST
- C12 pad 1: +5V -> +3V3
- C15 pad 1: Net-(C15-Pad1) -> +5V
- C2 pad 1: Net-(C2-Pad1) -> +3V3
- C3 pad 1: Net-(C3-Pad1) -> +3V3
- C4 pad 1: +5V -> +3V3
- C5 pad 1: +5V -> +3V3
- C6 pad 1: +5V -> +3V3
- C7 pad 1: Net-(C7-Pad1) -> +5V
- C8 pad 1: +5V -> Net-(C8-Pad1)
- C9 pad 1: +5V -> +3V3
- D34 pad 1: ROW5 -> Net-(D34-Pad1)
- D35 pad 1: ROW6 -> Net-(D35-Pad1)
- D36 pad 1: ROW7 -> Net-(D36-Pad1)
- D37 pad 1: ROW8 -> Net-(D37-Pad1)
- D38 pad 1: ROW9 -> Net-(D38-Pad1)
- D39 pad 1: ROW5 -> Net-(D39-Pad1)
- D40 pad 1: ROW6 -> Net-(D40-Pad1)
- D41 pad 1: ROW7 -> Net-(D41-Pad1)
- D42 pad 1: ROW8 -> Net-(D42-Pad1)
- D43 pad 1: ROW9 -> Net-(D43-Pad1)
- D44 pad 1: ROW5 -> Net-(D44-Pad1)
- D45 pad 1: ROW6 -> Net-(D45-Pad1)
- D46 pad 1: ROW7 -> Net-(D46-Pad1)
- D47 pad 1: ROW8 -> Net-(D47-Pad1)
- D48 pad 1: ROW9 -> Net-(D48-Pad1)
- D5 pad 1: ROW0 -> ROW2
- J1 pad 2: TRRS1 -> usart1
- J1 pad 3: TRRS0 -> +3V3
- J2 pad 2: TRRS1 -> usart1
- J2 pad 3: TRRS0 -> +3V3
- MX'1 pad 2: Net-(D61-Pad2) -> Net-(D46-Pad2)
- MX,1 pad 1: COL9 -> Net-(D42-Pad1)
- MX,1 pad 2: Net-(D47-Pad2) -> COL9
- MX.1 pad 2: Net-(D52-Pad2) -> Net-(D42-Pad2)
- MX/1 pad 1: COL11 -> Net-(D47-Pad1)
- MX/1 pad 2: Net-(D57-Pad2) -> COL11
- MX0 pad 1: COL11 -> Net-(D44-Pad1)
- MX0 pad 2: Net-(D54-Pad2) -> COL11
- MX6 pad 1: COL7 -> Net-(D34-Pad1)
- MX6 pad 2: Net-(D34-Pad2) -> COL7
- MX7 pad 2: Net-(D39-Pad2) -> Net-(D34-Pad2)
- MX8 pad 1: COL9 -> Net-(D39-Pad1)
- MX8 pad 2: Net-(D44-Pad2) -> COL9
- MX9 pad 2: Net-(D49-Pad2) -> Net-(D39-Pad2)
- MX;1 pad 1: COL11 -> Net-(D46-Pad1)
- MX;1 pad 2: Net-(D56-Pad2) -> COL11
- MX`-1 pad 2: Net-(D59-Pad2) -> Net-(D44-Pad2)
- MXdown1 pad 2: Net-(D53-Pad2) -> Net-(D43-Pad2)
- MXh1 pad 1: COL7 -> Net-(D36-Pad1)
- MXh1 pad 2: Net-(D36-Pad2) -> COL7
- MXi1 pad 1: COL9 -> Net-(D40-Pad1)
- MXi1 pad 2: Net-(D45-Pad2) -> COL9
- MXj1 pad 2: Net-(D41-Pad2) -> Net-(D36-Pad2)
- MXk1 pad 1: COL9 -> Net-(D41-Pad1)
- MXk1 pad 2: Net-(D46-Pad2) -> COL9
- MXl1 pad 2: Net-(D51-Pad2) -> Net-(D41-Pad2)
- MXleft1 pad 1: COL9 -> Net-(D43-Pad1)
- MXleft1 pad 2: Net-(D48-Pad2) -> COL9
- MXm1 pad 2: Net-(D42-Pad2) -> Net-(D37-Pad2)
- MXn1 pad 1: COL7 -> Net-(D37-Pad1)
- MXn1 pad 2: Net-(D37-Pad2) -> COL7
- MXo1 pad 2: Net-(D50-Pad2) -> Net-(D40-Pad2)
- MXp1 pad 1: COL11 -> Net-(D45-Pad1)
- MXp1 pad 2: Net-(D55-Pad2) -> COL11
- MXright1 pad 2: Net-(D63-Pad2) -> Net-(D48-Pad2)
- MXsh_r1 pad 2: Net-(D62-Pad2) -> Net-(D47-Pad2)
- MXsp_r0 pad 2: Net-(D38-Pad2) -> Net-(D38-Pad1)
- MXsp_r1 pad 2: Net-(D43-Pad2) -> Net-(D38-Pad2)
- MXsp_rC1 pad 2: Net-(D43-Pad2) -> Net-(D38-Pad2)
- MXtb[1 pad 2: Net-(D60-Pad2) -> Net-(D45-Pad2)
- MXu1 pad 2: Net-(D40-Pad2) -> Net-(D35-Pad2)
- MXup1 pad 1: COL11 -> Net-(D48-Pad1)
- MXup1 pad 2: Net-(D58-Pad2) -> COL11
- MXy1 pad 1: COL7 -> Net-(D35-Pad1)
- MXy1 pad 2: Net-(D35-Pad2) -> COL7
- R1 pad 1: TRRS1 -> +5V
- R1 pad 2: +5V -> GND
- R2 pad 1: TRRS0 -> usart1
- R2 pad 2: +5V -> +3V3
- R3 pad 1: +5V -> +3V3
- R3 pad 2: TRRS0 -> usart1
- R4 pad 1: +5V -> Net-(C8-Pad1)
- R4 pad 2: TRRS1 -> GND
- R5 pad 2: D- -> Net-(C39-Pad1)
- R6 pad 1: Net-(R6-Pad1) -> Net-(C42-Pad2)
- R6 pad 2: D+ -> Net-(C41-Pad2)
- R7 pad 1: +5V -> Net-(R7-Pad1)
- R7 pad 2: Net-(R7-Pad2) -> Net-(C43-Pad1)
- R8 pad 1: GND -> Net-(C46-Pad2)
- R8 pad 2: Net-(R8-Pad2) -> Net-(C45-Pad2)
- SW4 pad 1: GND -> +3V3
- SW4 pad 2: Net-(R7-Pad2) -> Net-(D21-Pad2)
- U1 pad 1: COL0 -> Net-(U1-Pad1)
- U1 pad 2: +5V -> LED3v
- U1 pad 3: Net-(R5-Pad1) -> GND
- U1 pad 4: Net-(R6-Pad1) -> LED5V
- U1 pad 5: GND -> +5V
- U2 pad 1: Net-(U2-Pad1) -> GND
- U2 pad 2: +5V -> +3V3
- U2 pad 3: Net-(R9-Pad1) -> +5V
- U3 pad 1: D- -> Net-(R5-Pad1)
- U3 pad 3: D- -> SPKR2
- U3 pad 4: D+ -> GND
- U3 pad 5: +5V -> Net-(C42-Pad2)
- U3 pad 6: D+ -> +5V
- U4 pad 1: TRRS0 -> +3V3
- U4 pad 3: TRRS0 -> +3V3
- U4 pad 4: TRRS1 -> usart1
- U4 pad 6: TRRS1 -> usart1
- U5 pad 1: TRRS0 -> +3V3
- U5 pad 3: TRRS0 -> +3V3
- U5 pad 4: TRRS1 -> usart1
- U5 pad 6: TRRS1 -> usart1
- U6 pad 1: D+ -> Net-(R7-Pad1)
- U6 pad 3: D+ -> SPKR2
- U6 pad 4: D- -> GND
- U6 pad 5: +5V -> Net-(C46-Pad2)
- U6 pad 6: D- -> +5V
Routing:
- net +3V3: track 0.00 -> 629.4 mm, vias 0 -> 24
- net GND: track 926.4 -> 358.9 mm, vias 59 -> 51
- net +5V: track 607.3 -> 116.5 mm, vias 19 -> 25
- net TRRS0: track 410.3 -> 0.00 mm, vias 11 -> 0
- net TRRS1: track 400.9 -> 0.00 mm, vias 10 -> 0
- net usart1: track 0.00 -> 350.4 mm, vias 0 -> 8
- net SWDIO: track 0.00 -> 107.2 mm, vias 0 -> 8
- net SWCLK: track 0.00 -> 105.5 mm, vias 0 -> 6
- net NRST: track 0.00 -> 99.5 mm, vias 0 -> 4
- net USART2_CTS: track 0.00 -> 87.7 mm, vias 0 -> 4
- net USART2_RX: track 0.00 -> 87.4 mm, vias 0 -> 4
- net USART2_CK: track 0.00 -> 87.0 mm, vias 0 -> 4
- net USART2_TX: track 0.00 -> 86.9 mm, vias 0 -> 4
- net USART2_RTS: track 0.00 -> 85.5 mm, vias 0 -> 4
- net LED3v3: track 0.00 -> 77.8 mm, vias 0 -> 4
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- added copper zone on F.Cu, net +5V
- removed copper zone on F.Cu, net GND
Other:
- net class Default: trace_width 0.254 -> 0.25; via_dia 0.8 -> 0.6; via_drill 0.4 -> 0.3
- net class Power: trace_width 0.381 -> 0.25; via_dia 0.8 -> 0.6; via_drill 0.4 -> 0.3
- net class USB added: clearance 0.2, trace_width 0.25, via_dia 0.6, via_drill 0.3

Commit message: Add shield grounding, curves etc
Parts:
- removed the H7 at (-110.7, 167.1)
- removed REF** (x2): Stabilizer_MX_2u, keyswitches:Stabilizer_MX_2u
- added C47: 4.7nF, Capacitor_SMD:C_0402_1005Metric, B.Cu at (-88.9, 115.9)
- added C48: 4.7nF, Capacitor_SMD:C_0402_1005Metric, B.Cu at (159.1, 114.7)
- added C49: 100nF, Capacitor_SMD:C_0402_1005Metric, B.Cu at (-99.4, 121.7)
- added C50: 100nF, Capacitor_SMD:C_0402_1005Metric, B.Cu at (173.4, 122.7)
- added H2: Hole, 3d-split-keeb:Mounting_Wuerth_WA-SMSI-M2_H3.5mm_9774035243, F.Cu at (-110.7, 167.1)
- added R10: 1M, Resistor_SMD:R_0402_1005Metric, B.Cu at (160.3, 114.7)
- added R9: 1M, Resistor_SMD:R_0402_1005Metric, B.Cu at (-90.1, 115.9)
- added STAB1: Hole, keyswitches:Stabilizer_MX_2u, F.Cu at (55.6, 199.2)
- added STAB2: Hole, keyswitches:Stabilizer_MX_2u, F.Cu at (17.5, 199.2)
- moved R15 1.19 mm to (161.9, 115.9)
- moved R16 0.79 mm to (179.0, 115.9)
- moved J5 0.40 mm to (-84.9, 117.9)
Connections:
- B2 pad 3: USART2_TX -> Net-(B2-Pad3)
- B2 pad 4: USART2_RX -> Net-(B2-Pad4)
- B2 pad 9: USART2_RTS -> Net-(B2-Pad9)
- H1 pad 1: (no net) -> GNDS
- H10 pad 1: (no net) -> GNDS
- H7 pad 1: (no net) -> GNDS
- H8 pad 1: (no net) -> GNDS
- J3 pad S1: Net-(J3-PadS1) -> GNDS
- J4 pad S1: Net-(J4-PadS1) -> GNDS
Routing:
- net GNDS: track 0.00 -> 538.7 mm, vias 0 -> 3
- net GND: track 358.9 -> 513.7 mm, vias 51 -> 61
- net ROW8: track 155.2 -> 196.3 mm
- net ROW6: track 157.8 -> 145.9 mm
- net Net-(D66-Pad2): track 11.7 -> 16.7 mm
- net NRST: track 99.5 -> 95.4 mm, vias 4 -> 6
- net VCC: track 50.9 -> 54.0 mm, vias 9 -> 11
- net SWCLK: track 105.5 -> 102.7 mm
- net +3V3: track 629.4 -> 632.0 mm
- net COL8: track 220.1 -> 222.6 mm
- net ROW9: track 177.5 -> 180.0 mm
- net Net-(J4-PadB5): track 11.4 -> 10.1 mm
- net Net-(D34-Pad2): track 15.7 -> 16.7 mm
- net Net-(J4-PadA5): track 9.33 -> 8.56 mm
Other:
- board size 320.7 x 98.5 mm -> 320.7 x 98.1 mm
- net class Power: trace_width 0.25 -> 0.375

Commit message: fix all the crossed labels
Connections:
- net LED3v3 renamed R_LED3v3
- B1 pad 12: SWCLK -> L_BT_SWCLK
- B1 pad 13: SWDIO -> L_BT_SWDIO
- B2 pad 10: USART2_RX -> R_USART2_RX
- B2 pad 11: USART2_TX -> R_USART2_TX
- B2 pad 12: SWCLK -> R_BT_SWCLK
- B2 pad 13: SWDIO -> R_BT_SWDIO
- B2 pad 14: USART2_CK -> R_USART2_CK
- B2 pad 15: USART2_CTS -> R_USART2_CTS
- B2 pad 18: USART2_RTS -> R_USART2_RTS
- C11 pad 1: NRST -> R_NRST
- C50 pad 1: VCC -> VCCQ
- D23 pad 4: LED5V -> R_LED5V
- F2 pad 2: VCC -> VCCQ
- J3 pad A6: D+ -> L_D+RAW
- J3 pad A7: D- -> L_D-RAW
- J3 pad B6: D+ -> L_D+RAW
- J3 pad B7: D- -> L_D-RAW
- J4 pad A4: VCC -> VCCQ
- J4 pad A6: D+ -> R_D+RAW
- J4 pad A7: D- -> R_D-RAW
- J4 pad A9: VCC -> VCCQ
- J4 pad B4: VCC -> VCCQ
- J4 pad B6: D+ -> R_D+RAW
- J4 pad B7: D- -> R_D-RAW
- J4 pad B9: VCC -> VCCQ
- J6 pad 2: SWDIO -> R_BT_SWDIO
- J6 pad 4: SWCLK -> R_BT_SWCLK
- J7 pad 10: NRST -> R_NRST
- J7 pad 2: SWDIO -> R_SWDIO
- J7 pad 4: SWCLK -> R_SWCLK
- J8 pad 2: SWDIO -> L_BT_SWDIO
- J8 pad 4: SWCLK -> L_BT_SWCLK
- Q2 pad 3: NRST -> R_NRST
- U10 pad 10: USART2_CTS -> R_USART2_CTS
- U10 pad 11: USART2_RTS -> R_USART2_RTS
- U10 pad 12: USART2_TX -> R_USART2_TX
- U10 pad 13: USART2_RX -> R_USART2_RX
- U10 pad 14: USART2_CK -> R_USART2_CK
- U10 pad 15: SPKR2 -> R_SPKR2
- U10 pad 32: D- -> R_D-
- U10 pad 33: D+ -> R_D+
- U10 pad 34: SWDIO -> R_SWDIO
- U10 pad 37: SWCLK -> R_SWCLK
- U10 pad 7: NRST -> R_NRST
- U11 pad 1: D- -> L_D-RAW
- U11 pad 3: D+ -> L_D+RAW
- U11 pad 4: D+ -> L_D+
- U11 pad 6: D- -> L_D-
- U12 pad 1: D- -> R_D-RAW
- U12 pad 3: D+ -> R_D+RAW
- U12 pad 4: D+ -> R_D+
- U12 pad 5: VCC -> VCCQ
- U12 pad 6: D- -> R_D-
- U6 pad 3: SPKR2 -> R_SPKR2
- U7 pad 32: D- -> L_D-
- U7 pad 33: D+ -> L_D+
- U8 pad 4: LED5V -> R_LED5V
Routing:
- net SWDIO: track 107.2 -> 17.1 mm, vias 8 -> 2
- net SWCLK: track 102.7 -> 15.3 mm, vias 6 -> 0
- net D-: track 68.0 -> 0.00 mm, vias 4 -> 0
- net D+: track 65.2 -> 0.00 mm, vias 4 -> 0
- net R_SWDIO: track 0.00 -> 57.4 mm, vias 0 -> 2
- net R_SWCLK: track 0.00 -> 53.5 mm, vias 0 -> 4
- net R_NRST: track 0.00 -> 53.1 mm, vias 0 -> 2
- net NRST: track 95.4 -> 42.3 mm, vias 6 -> 4
- net SPKR2: track 66.8 -> 26.7 mm, vias 4 -> 2
- net R_SPKR2: track 0.00 -> 40.1 mm, vias 0 -> 2
- net R_D-: track 0.00 -> 38.3 mm
- net R_D+: track 0.00 -> 37.9 mm
- net R_USART2_RX: track 0.00 -> 30.4 mm, vias 0 -> 2
- net USART2_RX: track 87.4 -> 56.9 mm, vias 4 -> 2
- net R_USART2_TX: track 0.00 -> 30.2 mm, vias 0 -> 2
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