File: basis_combined_PROTON.kicad_pcb (KiCad board)
At the start: 2 copper layers, 320.7 x 98.1 mm, 233 parts, among them J1 USB_B_Micro, J2 USB_B_Micro, J3 USB_C_Receptacle_USB2.0, J4 USB_C_Receptacle_USB2.0, J5 FTSH-105-01-L-DV-K, J6 FTSH-105-01-L-DV-K, J7 FTSH-105-01-L-DV-K, J8 FTSH-105-01-L-DV-K, Q1 DTC123J, Q2 DTC123J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

Commit message: shuffle the left amp
Parts:
- moved C41 8.11 mm to (-101.4, 168.6), turned to 0 degrees
- moved R6 5.43 mm to (-99.9, 168.1)
- moved C39 4.56 mm to (-105.0, 164.6)
- moved R5 4.56 mm to (-105.0, 162.1)
- moved U3 4.56 mm to (-101.8, 163.4)
- moved D6 4.55 mm to (-98.3, 143.5), turned to 225 degrees
- moved C40 4.53 mm to (-102.9, 167.6)
- moved D5 3.46 mm to (-99.3, 141.6), turned to 225 degrees
- moved C42 2.85 mm to (-98.8, 168.1), turned to 90 degrees
Routing:
- net ROW2: track 166.3 -> 159.3 mm
- net ROW4: track 170.2 -> 163.4 mm
- net ROW3: track 150.1 -> 145.6 mm
- net Net-(D6-Pad2): track 11.6 -> 14.1 mm
- net SPKR2: track 26.7 -> 24.6 mm
- net Net-(C42-Pad2): track 4.94 -> 2.83 mm
- net Net-(D5-Pad2): track 18.1 -> 19.9 mm
- net Net-(C42-Pad1): track 4.79 -> 6.55 mm
