File: basis_combined_PROTON.sch (KiCad schematic (older format))
At the start: 233 parts, among them J1 USB_B_Micro, J2 USB_B_Micro, J3 USB_C_Receptacle_USB2.0, J4 USB_C_Receptacle_USB2.0, J5 FTSH-105-01-L-DV-K, J6 FTSH-105-01-L-DV-K, J7 FTSH-105-01-L-DV-K, J8 FTSH-105-01-L-DV-K, Q1 DTC123J, Q2 DTC123J, SW1 Rotary_Encoder_Switch, SW2 Rotary_Encoder_Switch, SW3 Rotary_Encoder_Switch, SW4 SW_Push, SW6 SW_Push, U1 SN74LVC1G07DCK3, U10 STM32F072CBUx, U11 USBLC6-2SC6, U12 USBLC6-2SC6, U2 XC6206PxxxMR, U3 LM386, U4 SRV05-4, U5 SRV05-4, U6 LM386, U7 STM32F072CBUx, U8 SN74LVC1G07DCK3, U9 XC6206PxxxMR

Commit message: fix all the crossed labels
Connections:
- net LED5V: no longer D23.4 (DIN), U8.4 (Y)
- net NRST: no longer C11.1, J7.10, Q2.3 (C), U10.7 (NRST)
- net SPKR2: no longer U10.15 (PA5), U6.3 (+)
- net SWCLK: no longer B1.12 (DIO9), B2.12 (DIO9), J6.4, J7.4, J8.4, U10.37 (PA14)
- net SWDIO: no longer B1.13 (DIO10), B2.13 (DIO10), J6.2, J7.2, J8.2, U10.34 (PA13)
- net USART2_CK: no longer B2.14 (ANATEST1), U10.14 (PA4)
- net USART2_CTS: no longer B2.15 (DIO0), U10.10 (PA0)
- net USART2_RTS: no longer B2.18 (DIO1), U10.11 (PA1)
- net USART2_RX: no longer B2.10 (DIO8), U10.13 (PA3)
- net USART2_TX: no longer B2.11 (DIO11), U10.12 (PA2)
- net VCC: no longer C50.1, F2.2, J4.A4 (VBUS), J4.A9 (VBUS), J4.B4 (VBUS), J4.B9 (VBUS), U12.5 (VBUS)
- removed net D+: J3.A6 (D+), J3.B6 (D+), J4.A6 (D+), J4.B6 (D+), U10.33 (PA12), U11.3 (IO2), U11.4 (IO2), U12.3 (IO2), U12.4 (IO2), U7.33 (PA12)
- removed net D-: J3.A7 (D-), J3.B7 (D-), J4.A7 (D-), J4.B7 (D-), U10.32 (PA11), U11.1 (IO1), U11.6 (IO1), U12.1 (IO1), U12.6 (IO1), U7.32 (PA11)
- net LED3v3 renamed R_LED3v3
- new net L_BT_SWCLK: B1.12 (DIO9), J8.4
- new net L_BT_SWDIO: B1.13 (DIO10), J8.2
- new net L_D+: U11.4 (IO2), U7.33 (PA12)
- new net L_D+RAW: J3.A6 (D+), J3.B6 (D+), U11.3 (IO2)
- new net L_D-: U11.6 (IO1), U7.32 (PA11)
- new net L_D-RAW: J3.A7 (D-), J3.B7 (D-), U11.1 (IO1)
- new net R_BT_SWCLK: B2.12 (DIO9), J6.4
- new net R_BT_SWDIO: B2.13 (DIO10), J6.2
- new net R_D+: U10.33 (PA12), U12.4 (IO2)
- new net R_D+RAW: J4.A6 (D+), J4.B6 (D+), U12.3 (IO2)
- new net R_D-: U10.32 (PA11), U12.6 (IO1)
- new net R_D-RAW: J4.A7 (D-), J4.B7 (D-), U12.1 (IO1)
- new net R_LED5V: D23.4 (DIN), U8.4 (Y)
- new net R_NRST: C11.1, J7.10, Q2.3 (C), U10.7 (NRST)
- new net R_SPKR2: U10.15 (PA5), U6.3 (+)
- new net R_SWCLK: J7.4, U10.37 (PA14)
- new net R_SWDIO: J7.2, U10.34 (PA13)
- new net R_USART2_CK: B2.14 (ANATEST1), U10.14 (PA4)
- new net R_USART2_CTS: B2.15 (DIO0), U10.10 (PA0)
- new net R_USART2_RTS: B2.18 (DIO1), U10.11 (PA1)
- new net R_USART2_RX: B2.10 (DIO8), U10.13 (PA3)
- new net R_USART2_TX: B2.11 (DIO11), U10.12 (PA2)
- new net VCCQ: C50.1, F2.2, J4.A4 (VBUS), J4.A9 (VBUS), J4.B4 (VBUS), J4.B9 (VBUS), U12.5 (VBUS)
Other:
- moved on the sheet: C49, C50, F1, F2, U11, U12
Changed lines of the file:
@@
 L Device:Polyfuse_Small F1
 U 1 1 5F2E04FA
-P 13300 1000
-F 0 "F1" V 13095 1000 50  0000 C CNN
-F 1 "500mA" V 13186 1000 50  0000 C CNN
-F 2 "Fuse:Fuse_1206_3216Metric" H 13350 800 50  0001 L CNN
-F 3 "~" H 13300 1000 50  0001 C CNN
-	1    13300 1000
+P 13500 7550
+F 0 "F1" V 13295 7550 50  0000 C CNN
+F 1 "500mA" V 13386 7550 50  0000 C CNN
+F 2 "Fuse:Fuse_1206_3216Metric" H 13550 7350 50  0001 L CNN
+F 3 "~" H 13500 7550 50  0001 C CNN
+	1    13500 7550
 	0    1    1    0
 $EndComp
@@
 L Device:Polyfuse_Small F2
 U 1 1 5F66D4D9
-P 13500 7550
-F 0 "F2" V 13295 7550 50  0000 C CNN
-F 1 "500mA" V 13386 7550 50  0000 C CNN
-F 2 "Fuse:Fuse_1206_3216Metric" H 13550 7350 50  0001 L CNN
-F 3 "~" H 13500 7550 50  0001 C CNN
-	1    13500 7550
+P 13300 1000
+F 0 "F2" V 13095 1000 50  0000 C CNN
+F 1 "500mA" V 13186 1000 50  0000 C CNN
+F 2 "Fuse:Fuse_1206_3216Metric" H 13350 800 50  0001 L CNN
+F 3 "~" H 13300 1000 50  0001 C CNN
+	1    13300 1000
 	0    1    1    0
 $EndComp
 Text GLabel 8050 9350 0    50   Input ~ 0
-LED3v3
+R_LED3v3
 Text GLabel 8150 8950 0    50   Input ~ 0
 COL13
@@
 	1    0    0    -1
 $EndComp
-Wire Wire Line
-	12500 1000 13000 1000
 $Comp
 L power:+5V #PWR0116
@@
 Wire Wire Line
 	13400 1000 13550 1000
-$Comp
-L power:VCC #PWR0117
-U 1 1 612CF0B3
-P 13000 1000
-F 0 "#PWR0117" H 13000 850 50  0001 C CNN
-F 1 "VCC" H 13017 1173 50  0000 C CNN
-F 2 "" H 13000 1000 50  0001 C CNN
-F 3 "" H 13000 1000 50  0001 C CNN
-	1    13000 1000
-	1    0    0    -1
-$EndComp
-Connection ~ 13000 1000
-Wire Wire Line
-	13000 1000 13200 1000
 Text GLabel 14150 1350 2    50   Input ~ 0
-D-
+R_D-
 Text GLabel 14150 2350 2    50   Input ~ 0
-D+
+R_D+
 $Comp
 L power:GND #PWR0136
@@
 $EndComp
 Text GLabel 13900 7950 2    50   Input ~ 0
-D-
+L_D-
 Text GLabel 13900 8950 2    50   Input ~ 0
-D+
+L_D+
 $Comp
 L power:GND #PWR0139
@@
 $EndComp
 Text GLabel 2650 4450 2    50   Input ~ 0
-D-
+L_D-
 Text GLabel 2650 4550 2    50   Input ~ 0
-D+
+L_D+
 Wire Wire Line
 	2500 4450 2650 4450
@@
 $EndComp
 Text GLabel 9600 9650 2    50   Input ~ 0
-D-
+R_D-
 Text GLabel 9600 9750 2    50   Input ~ 0
-D+
+R_D+
 Wire Wire Line
 	9450 9650 9600 9650
@@
 	9450 9050 9600 9050
 Text GLabel 9600 9050 2    50   Input ~ 0
-SPKR2
+R_SPKR2
 Text GLabel 8700 5850 0    50   Input ~ 0
-LED3v3
+R_LED3v3
 $Comp
 L Regulator_Linear:XC6206PxxxMR U2
@@
 	9450 8750 9600 8750
 Text GLabel 9600 8750 2    50   Input ~ 0
-USART2_TX
+R_USART2_TX
 Wire Wire Line
 	9450 9850 9550 9850
 Text GLabel 9550 9850 2    50   Input ~ 0
-SWDIO
+R_SWDIO
 Wire Wire Line
 	9450 9950 9550 9950
 Text GLabel 9550 9950 2    50   Input ~ 0
-SWCLK
+R_SWCLK
 Wire Wire Line
 	7100 9650 7100 9950
@@
 $EndComp
 Text GLabel 10900 5850 2    50   Input ~ 0
-LED5V
+R_LED5V
 $Comp
 L SN74LVC1G07DCKR:SN74LVC1G07DCK3 U8
@@
 	11200 10350 11250 10350
 Text GLabel 11250 10350 2    50   Input ~ 0
-NRST
+R_NRST
 $Comp
 L power:GND #PWR0130
@@
 	11200 10050 11250 10050
 Text GLabel 11250 10050 2    50   Input ~ 0
-SWCLK
+R_SWCLK
 $Comp
 L FTSH-105-01-L-DV-K:FTSH-105-01-L-DV-K J7
@@
 	11200 9950 11250 9950
 Text GLabel 11250 9950 2    50   Input ~ 0
-SWDIO
+R_SWDIO
 Wire Wire Line
 	10400 9950 10350 9950
@@
 	1250 11750 1100 11750
 Text GLabel 1100 11750 0    50   Input ~ 0
-LED5V
+R_LED5V
 Wire Wire Line
 	1850 11750 2200 11750
@@
 L Power_Protection:USBLC6-2SC6 U11
 U 1 1 66C253CB
-P 13450 1850
-F 0 "U11" H 13450 2531 50  0000 C CNN
-F 1 "USBLC6-2SC6" H 13450 2440 50  0000 C CNN
-F 2 "Package_TO_SOT_SMD:SOT-666" H 12700 2250 50  0001 C CNN
-F 3 "http://www2.st.com/resource/en/datasheet/CD00050750.pdf" H 13650 2200 50  0001 C CNN
-	1    13450 1850
-	0    1    1    0
-$EndComp
-$Comp
-L Power_Protection:USBLC6-2SC6 U12
-U 1 1 66C2D08D
 P 13500 8450
-F 0 "U12" H 13500 9131 50  0000 C CNN
+F 0 "U11" H 13500 9131 50  0000 C CNN
 F 1 "USBLC6-2SC6" H 13500 9040 50  0000 C CNN
 F 2 "Package_TO_SOT_SMD:SOT-666" H 12750 8850 50  0001 C CNN
@@
 	0    1    1    0
 $EndComp
-Wire Wire Line
-	12950 7950 13400 7950
 $Comp
-L power:VCC #PWR0125
-U 1 1 673C13A2
-P 14650 1850
-F 0 "#PWR0125" H 14650 1700 50  0001 C CNN
-F 1 "VCC" H 14667 2023 50  0000 C CNN
-F 2 "" H 14650 1850 50  0001 C CNN
-F 3 "" H 14650 1850 50  0001 C CNN
-	1    14650 1850
-	1    0    0    -1
+L Power_Protection:USBLC6-2SC6 U12
+U 1 1 66C2D08D
+P 13450 1850
+F 0 "U12" H 13450 2531 50  0000 C CNN
+F 1 "USBLC6-2SC6" H 13450 2440 50  0000 C CNN
+F 2 "Package_TO_SOT_SMD:SOT-666" H 12700 2250 50  0001 C CNN
+F 3 "http://www2.st.com/resource/en/datasheet/CD00050750.pdf" H 13650 2200 50  0001 C CNN
+	1    13450 1850
+	0    1    1    0
 $EndComp
+Wire Wire Line
+	12950 7950 13400 7950
 $Comp
 L power:VCC #PWR0133
@@
 	9450 8650 9600 8650
 Text GLabel 9600 8650 2    50   Input ~ 0
-USART2_RTS
+R_USART2_RTS
 Wire Wire Line
 	9450 8550 9600 8550
 Text GLabel 9600 8550 2    50   Input ~ 0
-USART2_CTS
+R_USART2_CTS
 Wire Wire Line
 	9450 8850 9600 8850
 Text GLabel 9600 8850 2    50   Input ~ 0
-USART2_RX
+R_USART2_RX
 Text GLabel 9600 8950 2    50   Input ~ 0
-USART2_CK
+R_USART2_CK
 Wire Wire Line
 	9700 11500 9800 11500
@@
 	9700 11100 9800 11100
 Text GLabel 9800 11100 2    50   Input ~ 0
-USART2_CTS
+R_USART2_CTS
 Text GLabel 9700 12150 2    50   Input ~ 0
-USART2_TX
+R_USART2_TX
 Text GLabel 9700 11850 2    50   Input ~ 0
-USART2_RX
+R_USART2_RX
 Wire Wire Line
 	9700 11700 9800 11700
 Text GLabel 9700 11200 2    50   Input ~ 0
-USART2_RTS
+R_USART2_RTS
 $Comp
 L Amplifier_Audio:LM386 U3
@@
 	5600 5800 5400 5800
 Text GLabel 5400 5800 0    50   Input ~ 0
-SPKR2
+R_SPKR2
 $Comp
 L power:GND #PWR0160
@@
 	9700 11950 10200 11950
 Text GLabel 10200 11950 2    50   Input ~ 0
-SWCLK
+R_BT_SWCLK
 Wire Wire Line
 	9700 12050 10200 12050
 Text GLabel 10200 12050 2    50   Input ~ 0
-SWDIO
+R_BT_SWDIO
 $Comp
 L power:GND #PWR0163
@@
 	8000 10800 8050 10800
 Text GLabel 8050 10800 2    50   Input ~ 0
-SWCLK
+R_BT_SWCLK
 $Comp
 L FTSH-105-01-L-DV-K:FTSH-105-01-L-DV-K J6
@@
 	8000 10700 8050 10700
 Text GLabel 8050 10700 2    50   Input ~ 0
-SWDIO
+R_BT_SWDIO
 Wire Wire Line
 	7100 10700 7200 10700
@@
 	8500 11850 8400 11850
 Text GLabel 8400 11850 0    50   Input ~ 0
-USART2_CK
+R_USART2_CK
 $Comp
 L power:+3.3V #PWR0167
@@
 $EndComp
 Text GLabel 8150 7250 2    50   Input ~ 0
-NRST
+R_NRST
 Wire Wire Line
 	8150 7450 8100 7450
 Text GLabel 8100 7450 0    50   Input ~ 0
-NRST
+R_NRST
 Connection ~ 8950 7250
 Connection ~ 8850 7250
@@
 	-2000 5850 -1950 5850
 Text GLabel -1950 5850 2    50   Input ~ 0
-SWCLK
+L_BT_SWCLK
 $Comp
 L FTSH-105-01-L-DV-K:FTSH-105-01-L-DV-K J8
@@
 	-2000 5750 -1950 5750
 Text GLabel -1950 5750 2    50   Input ~ 0
-SWDIO
+L_BT_SWDIO
 Wire Wire Line
 	-2900 5750 -2800 5750
@@
 	-300 7000 200  7000
 Text GLabel 200  7000 2    50   Input ~ 0
-SWCLK
+L_BT_SWCLK
 Wire Wire Line
 	-300 7100 200  7100
 Text GLabel 200  7100 2    50   Input ~ 0
-SWDIO
+L_BT_SWDIO
 Text GLabel -200 6750 2    50   Input ~ 0
 USART2_RTS
@@
 	13600 8950 13900 8950
 Text GLabel 13100 7950 1    50   Input ~ 0
-D-
+L_D-RAW
 Text GLabel 13050 8950 3    50   Input ~ 0
-D+
+L_D+RAW
 Text GLabel 13100 1350 1    50   Input ~ 0
-D-
+R_D-RAW
 Text GLabel 13050 2350 3    50   Input ~ 0
-D+
+R_D+RAW
 $Comp
 L Device:C_Small C49
 U 1 1 6544880F
-P 14350 1950
-F 0 "C49" H 14442 1996 50  0000 L CNN
-F 1 "100nF" H 14442 1905 50  0000 L CNN
-F 2 "Capacitor_SMD:C_0402_1005Metric" H 14350 1950 50  0001 C CNN
-F 3 "~" H 14350 1950 50  0001 C CNN
-	1    14350 1950
+P 14350 8550
+F 0 "C49" H 14442 8596 50  0000 L CNN
+F 1 "100nF" H 14442 8505 50  0000 L CNN
+F 2 "Capacitor_SMD:C_0402_1005Metric" H 14350 8550 50  0001 C CNN
+F 3 "~" H 14350 8550 50  0001 C CNN
+	1    14350 8550
 	1    0    0    -1
 $EndComp
 Wire Wire Line
-	13950 1850 14350 1850
+	13950 1850 14250 1850
 Connection ~ 14350 1850
 Wire Wire Line
@@
 	12950 1850 12950 2050
 Wire Wire Line
-	12950 2050 14350 2050
+	12950 2050 14250 2050
 Connection ~ 14350 2050
 Wire Wire Line
@@
 L Device:C_Small C50
 U 1 1 6554BD4E
-P 14350 8550
-F 0 "C50" H 14442 8596 50  0000 L CNN
-F 1 "100nF" H 14442 8505 50  0000 L CNN
-F 2 "Capacitor_SMD:C_0402_1005Metric" H 14350 8550 50  0001 C CNN
-F 3 "~" H 14350 8550 50  0001 C CNN
-	1    14350 8550
+P 14250 1950
+F 0 "C50" H 14342 1996 50  0000 L CNN
+F 1 "100nF" H 14342 1905 50  0000 L CNN
+F 2 "Capacitor_SMD:C_0402_1005Metric" H 14250 1950 50  0001 C CNN
+F 3 "~" H 14250 1950 50  0001 C CNN
+	1    14250 1950
 	1    0    0    -1
 $EndComp
@@
 	14350 8650 14650 8650
 $Comp
-L power:GNDS #PWR?
+L power:GNDS #PWR0182
 U 1 1 65697079
 P 10500 1100
-F 0 "#PWR?" H 10500 850 50  0001 C CNN
+F 0 "#PWR0182" H 10500 850 50  0001 C CNN
 F 1 "GNDS" V 10505 972 50  0000 R CNN
 F 2 "" H 10500 1100 50  0001 C CNN
@@
 $EndComp
 $Comp
-L power:GNDS #PWR?
+L power:GNDS #PWR0183
 U 1 1 656976B2
 P 11150 1650
-F 0 "#PWR?" H 11150 1400 50  0001 C CNN
+F 0 "#PWR0183" H 11150 1400 50  0001 C CNN
 F 1 "GNDS" V 11155 1522 50  0000 R CNN
 F 2 "" H 11150 1650 50  0001 C CNN
@@
 	0    -1   -1   0
 $EndComp
+$Comp
+L power:VCCQ #PWR0117
+U 1 1 6578B369
+P 12900 1000
+F 0 "#PWR0117" H 12900 850 50  0001 C CNN
+F 1 "VCCQ" H 12917 1173 50  0000 C CNN
+F 2 "" H 12900 1000 50  0001 C CNN
+F 3 "" H 12900 1000 50  0001 C CNN
+	1    12900 1000
+	1    0    0    -1
+$EndComp
+Wire Wire Line
+	12500 1000 12900 1000
+Connection ~ 12900 1000
+Wire Wire Line
+	12900 1000 13200 1000
+$Comp
+L power:VCCQ #PWR0125
+U 1 1 6591E530
+P 14650 1850
+F 0 "#PWR0125" H 14650 1700 50  0001 C CNN
+F 1 "VCCQ" H 14667 2023 50  0000 C CNN
+F 2 "" H 14650 1850 50  0001 C CNN
+F 3 "" H 14650 1850 50  0001 C CNN
+	1    14650 1850
+	1    0    0    -1
+$EndComp
+Connection ~ 14250 1850
+Wire Wire Line
+	14250 1850 14350 1850
+Connection ~ 14250 2050
+Wire Wire Line
+	14250 2050 14350 2050
 $EndSCHEMATC

Commit message: v2!
Parts:
- removed H9: Hole, 3d-split-keeb:Mounting_Wuerth_WA-SMSI-M2_H3.5mm_9774035243, symbol keebio:Hole
- added C51, C52, C55, C56: 100uF, Capacitor_SMD:C_1206_3216Metric, symbol Device:C_Small
- added C53: 47uF, Capacitor_SMD:C_1206_3216Metric, symbol Device:C_Small
- added C54: 33nF, Capacitor_SMD:C_0402_1005Metric, symbol Device:C_Small
- added R11, R12: 33k, Resistor_SMD:R_0402_1005Metric, symbol Device:R_Small
- C20: value 10nF -> 100uF
- C40, C44: value 50uF -> 100nF
- C41, C45: value 50nF -> 22nF
- C42: value 250uF -> 33nF
- C46: value 250uF -> 47uF; footprint Capacitor_SMD:C_0402_1005Metric -> Capacitor_SMD:C_1206_3216Metric
- C8: value 10nF -> 100uF; footprint Capacitor_SMD:C_0402_1005Metric -> Capacitor_SMD:C_1206_3216Metric
- D1, D14, D2, D9: LCSC (none) -> C375703
Connections:
- net GND: now also C42.1, C54.1
- net at R6.1, U3.5: now also C51.2, C52.2, C53.2; no longer C42.2
- net at LS1.1: now also C51.1, C52.1, C53.1; no longer C42.1
- net at C41.2, R6.2: now also C42.2
- net at C46.2, R8.1, U6.5: now also C55.2, C56.2
- net at C46.1, LS2.1: now also C55.1, C56.1
- net at C45.2, R8.2: now also C54.2
- net at C20.1, R17.1, U7.44 (BOOT0): now also R11.2; no longer D19.1 (K)
- net at C8.1, R4.1, U10.44 (BOOT0): now also R12.1; no longer D21.1 (K)
- new net: D19.1 (K), R11.1
- new net: D21.1 (K), R12.2
Other:
- moved on the sheet: B1, B2, C1, C10, C11, C12, C13, C14, C15, C16, C17, C18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
