File: basis_combined_PROTON.sch (KiCad schematic (older format))
At the start: 240 parts, among them J1 USB_B_Micro, J2 USB_B_Micro, J3 USB_C_Receptacle_USB2.0, J4 USB_C_Receptacle_USB2.0, J5 FTSH-105-01-L-DV-K, J6 FTSH-105-01-L-DV-K, J7 FTSH-105-01-L-DV-K, J8 FTSH-105-01-L-DV-K, Q1 DTC123J, Q2 DTC123J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

Commit message: v3 gerbers
Parts:
- removed B1, B2: BLUENRG-M2SA, 3d-split-keeb:BLUENRG-M2SA, symbol random-keyboard-parts:BLUENRG-M2SA
- removed C43: 10uF, Capacitor_SMD:C_0402_1005Metric, symbol Device:C_Small
- removed C44, C49, C50: 100nF, Capacitor_SMD:C_0402_1005Metric, symbol Device:C_Small
- removed C45: 22nF, Capacitor_SMD:C_0402_1005Metric, symbol Device:C_Small
- removed C46, C53: 47uF, Capacitor_SMD:C_1206_3216Metric, symbol Device:C_Small
- removed C51, C52, C55, C56: 100uF, Capacitor_SMD:C_1206_3216Metric, symbol Device:C_Small
- removed C54: 33nF, Capacitor_SMD:C_0402_1005Metric, symbol Device:C_Small
- removed H10, H8: Hole, 3d-split-keeb:Mounting_Wuerth_WA-SMSI-M2_H3.5mm_9774035243, symbol keebio:eHole
- removed J6, J8: FTSH-105-01-L-DV-K, FTSH-105-01-L-DV-K:SAMTEC_FTSH-105-01-L-DV-K, symbol FTSH-105-01-L-DV-K:FTSH-105-01-L-DV-K
- removed R7: 1.2k, Resistor_SMD:R_0402_1005Metric, symbol Device:R_Small
- removed R8: 10, Resistor_SMD:R_0402_1005Metric, symbol Device:R_Small
- removed U10, U7: STM32F072CBUx, Package_DFN_QFN:QFN-48-1EP_7x7mm_P0.5mm_EP5.6x5.6mm, symbol MCU_ST_STM32F0:STM32F072CBUx
- removed U11, U12: USBLC6-2SC6, Package_TO_SOT_SMD:SOT-666, symbol Power_Protection:USBLC6-2SC6
- removed U3, U6: LM386, Package_SO:SOIC-8_3.9x4.9mm_P1.27mm, symbol Amplifier_Audio:LM386
- added D49, D50: WS2812B, LED_SMD:LED_WS2812B_PLCC4_5.0x5.0mm_P3.2mm, symbol LED:WS2812B
- added U10, U7: SRV05-4, Package_TO_SOT_SMD:SOT-23-6, symbol Power_Protection:SRV05-4
- added U3, U6: STM32L452CEUx, Package_DFN_QFN:QFN-48-1EP_7x7mm_P0.5mm_EP5.6x5.6mm, symbol MCU_ST_STM32L4:STM32L452CEUx
- C19, C3: value 4.7uF -> 1uF
- C20, C8: value 100uF -> 4.7uF
- C39: value 10uF -> 100nF
- C41: value 22nF -> 100nF
- C42: value 33nF -> 100nF
- D19, D21: value 1N4148 -> D_Small
- R5: value 1.2k -> 4.7k
- R6: value 10 -> 4.7k
- U1, U8: value SN74LVC1G07DCK3 -> SN74LV1T34DCKR
Connections:
- net labels added: BOOT0, R_BOOT0
- net labels removed: L_BT_SWCLK, L_BT_SWDIO, L_D+RAW, L_D-RAW, R_BT_SWCLK, R_BT_SWDIO, R_D+RAW, R_D-RAW, R_USART2_CK, R_USART2_CTS, R_USART2_RTS, R_USART2_RX, R_USART2_TX, USART2_CK, USART2_CTS, USART2_RTS, USART2_RX, USART2_TX
- wire segments 666 -> 580
Other:
- moved on the sheet: C30, C32, C34, C36, C37, C38, C47, D28, D30, D32, D69, D70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
